File: Feather_STM32WB55.sch (KiCad schematic (older format))
At the start: 44 parts, among them J1 JST-SH Qwiic, J2 Conn_Battery, J3 Conn_ARM_JTAG_SWD_10, J4 Conn_Right, J5 USB_C_Receptacle_USB2.0, J6 Conn_Left, Q1 NTR4171PT1G, SW1 SMD-BUTTON-TOP-DHT-4235A_4P-4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, U1 MCP73831-2-OT, U2 AP2112K-3.3, U3 STM32WB55CGU6, U4 USBLC6-2SC6, U5 Flash SOIC-8, Y1 32Mhz

Commit message: Updated with the matching network and antenna
Parts:
- removed AE1: Fractus NN01-102, DigiKey_Footprints:Antenna_1.6x3.2mm_2450AT18A100E, symbol Device:Antenna_Chip
- added ANT1: NN01-102, FR05S1N0102, symbol Makeristic-KiCad-Library:FR05-S1-N-0-102
- added FL1: MLPF-WB55-01E3, MLPFWB5501E3, symbol Makeristic-KiCad-Library:MLPF-WB55-01E3
- C5: footprint Capacitor_SMD:C_0805_2012Metric -> Capacitor_SMD:C_0603_1608Metric
- D1, D4: footprint LED_SMD:LED_0603_1608Metric_Pad1.05x0.95mm_HandSolder -> LED_SMD:LED_0603_1608Metric
- D3: footprint LED_SMD:LED_WS2812B_PLCC4_5.0x5.0mm_P3.2mm -> LED_SMD:LED_SK6812MINI_PLCC4_3.5x3.5mm_P1.75mm
- L1: footprint Inductor_SMD:L_0603_1608Metric_Pad1.05x0.95mm_HandSolder -> Inductor_SMD:L_0603_1608Metric
Connections:
- net labels added: ANT_OUT, RF_OUT
- wire segments 152 -> 151
- no-connect marks 9 -> 10
Other:
- moved on the sheet: C1, D1, J1, J5, R1, R2, R3, R7, R8, R9, U1, U4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
